Commit message: Add files via upload

File: robot.urdf (robot description, URDF)
Before this commit: robot onshape, 3 links, 2 joints
Links:
- removed link assembly_1_1
- removed link lego_motors:_small_angular_motor_1
- removed link lego_motors:_small_angular_motor_2
- added link body_sub_1, mass 0.204762; collision mesh filename=package://electric,_hub_-_spike_prime.stl; collision mesh filename=package://electric,_motor_small_angular_-_spike_prime-_axle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
Joints:
- removed joint 0782b20d-41d2-494e-b69c-b40690af0f38_fixing
- removed joint 38626c1f-f753-45d4-956d-35b5b2eb7e09_fixing
